File: design-files/register-module/register-module.sch (KiCad schematic (older format))
At the start: 106 parts, among them U201 74HCT377, U202 74HCT245, U203 AT28C64, U204 WL-T7DS-157136V12701, U205 WL-T7DS-157136V12701, U206 WL-T7DS-157136V12701, U207 WL-T7DS-157136V12701, U208 74HCT139, U209 74HCT377, U210 74HCT245, U211 AT28C64, U212 WL-T7DS-157136V12701, U213 WL-T7DS-157136V12701, U214 WL-T7DS-157136V12701, U215 WL-T7DS-157136V12701, U216 74HCT377, U217 74HCT245, U218 AT28C64, U219 WL-T7DS-157136V12701, U220 WL-T7DS-157136V12701, U221 WL-T7DS-157136V12701, U222 WL-T7DS-157136V12701, U223 74HCT139, U224 74HCT377, U225 74HCT245, U226 AT28C64, U227 WL-T7DS-157136V12701, U228 WL-T7DS-157136V12701, U229 WL-T7DS-157136V12701, U230 WL-T7DS-157136V12701, U231 74HCT161, U232 NE555P

Commit message: Annotate for resistor packs.
Parts:
- gave numbers to parts that had none: 6
Connections:
- net GND: now also RN204.1 (R1.1), RN204.2 (R2.1), RN204.3 (R3.1), RN204.4 (R4.1), RN204.5 (R5.1), RN204.6 (R6.1), RN204.7 (R7.1), RN204.8 (R8.1)
- net at U207.3 (CC), U207.8 (CC): now also RN202.12 (R5.2); no longer RN202.13 (R4.2)
- net at U206.3 (CC), U206.8 (CC): now also RN202.16 (R1.2); no longer RN202.14 (R3.2)
- net at U205.3 (CC), U205.8 (CC): now also RN201.12 (R5.2); no longer RN201.15 (R2.2)
- net at U208.5 (O1): now also RN201.5 (R5.1); no longer RN201.2 (R2.1)
- net at U208.6 (O2): now also RN202.1 (R1.1); no longer RN202.3 (R3.1)
- net at U208.7 (O3): now also RN202.5 (R5.1); no longer RN202.4 (R4.1)
- net at U215.3 (CC), U215.8 (CC): now also RN202.11 (R6.2); no longer RN202.9 (R8.2)
- net at U214.3 (CC), U214.8 (CC): now also RN202.15 (R2.2); no longer RN202.10 (R7.2)
- net at U212.3 (CC), U212.8 (CC): now also RN201.15 (R2.2); no longer RN201.12 (R5.2)
- net at U208.10 (O2): now also RN202.2 (R2.1); no longer RN202.7 (R7.1)
- net at U208.12 (O0): now also RN201.2 (R2.1); no longer RN201.5 (R5.1)
- net at U208.9 (O3): now also RN202.6 (R6.1); no longer RN202.8 (R8.1)
- net at U222.3 (CC), U222.8 (CC): now also RN202.10 (R7.2); no longer RN202.13 (R4.2)
- net at U220.3 (CC), U220.8 (CC): now also RN201.10 (R7.2); no longer RN201.15 (R2.2)
- net at U219.3 (CC), U219.8 (CC): now also RN201.14 (R3.2); no longer RN201.16 (R1.2)
- net at U223.4 (O0): now also RN201.3 (R3.1); no longer RN201.1 (R1.1)
- net at U223.5 (O1): now also RN201.7 (R7.1); no longer RN201.2 (R2.1)
- net at U223.7 (O3): now also RN202.7 (R7.1); no longer RN202.4 (R4.1)
- net at U229.3 (CC), U229.8 (CC): now also RN202.13 (R4.2); no longer RN202.10 (R7.2)
- net at U228.3 (CC), U228.8 (CC): now also RN201.9 (R8.2); no longer RN201.11 (R6.2)
- net at U227.3 (CC), U227.8 (CC): now also RN201.13 (R4.2); no longer RN201.12 (R5.2)
- net at U223.10 (O2): now also RN202.4 (R4.1); no longer RN202.7 (R7.1)
- net at U223.11 (O1): now also RN201.8 (R8.1); no longer RN201.6 (R6.1)
- net at U223.12 (O0): now also RN201.4 (R4.1); no longer RN201.5 (R5.1)
Changed lines of the file:
@@
 Nominal frequency: 718 Hz
 $Comp
-L Device:R_Pack08 RN?
+L Device:R_Pack08 RN203
 U 1 1 61EB3C65
 P 12550 1550
-F 0 "RN?" H 12938 1596 50  0000 L CNN
+F 0 "RN203" H 12938 1596 50  0000 L CNN
 F 1 "330 x 8" H 12938 1505 50  0000 L CNN
 F 2 "Package_DIP:DIP-16_W7.62mm_Socket" V 13025 1550 50  0001 C CNN
@@
 	13900 1050 13900 1350
 $Comp
-L power:GND #PWR?
+L power:GND #PWR0131
 U 1 1 62651987
-P 13050 3400
-F 0 "#PWR?" H 13050 3150 50  0001 C CNN
-F 1 "GND" H 13055 3227 50  0000 C CNN
-F 2 "" H 13050 3400 50  0001 C CNN
-F 3 "" H 13050 3400 50  0001 C CNN
-	1    13050 3400
-	1    0    0    -1
-$EndComp
-$Comp
-L Device:R_Pack08 RN?
+P 12850 3400
+F 0 "#PWR0131" H 12850 3150 50  0001 C CNN
+F 1 "GND" H 12855 3227 50  0000 C CNN
+F 2 "" H 12850 3400 50  0001 C CNN
+F 3 "" H 12850 3400 50  0001 C CNN
+	1    12850 3400
+	1    0    0    -1
+$EndComp
+$Comp
+L Device:R_Pack08 RN204
 U 1 1 6265198E
 P 12550 3200
-F 0 "RN?" H 12938 3246 50  0000 L CNN
+F 0 "RN204" H 12938 3246 50  0000 L CNN
 F 1 "330 x 8" H 12938 3155 50  0000 L CNN
 F 2 "Package_DIP:DIP-16_W7.62mm_Socket" V 13025 3200 50  0001 C CNN
@@
 	13900 2650 13900 3000
 $Comp
-L power:GND #PWR?
+L power:GND #PWR0132
 U 1 1 627313CF
 P 12850 5050
-F 0 "#PWR?" H 12850 4800 50  0001 C CNN
+F 0 "#PWR0132" H 12850 4800 50  0001 C CNN
 F 1 "GND" H 12855 4877 50  0000 C CNN
 F 2 "" H 12850 5050 50  0001 C CNN
@@
 $EndComp
 $Comp
-L Device:R_Pack08 RN?
+L Device:R_Pack08 RN205
 U 1 1 627313D6
 P 12550 4850
-F 0 "RN?" H 12938 4896 50  0000 L CNN
+F 0 "RN205" H 12938 4896 50  0000 L CNN
 F 1 "330 x 8" H 12938 4805 50  0000 L CNN
 F 2 "Package_DIP:DIP-16_W7.62mm_Socket" V 13025 4850 50  0001 C CNN
@@
 	13900 4300 13900 4650
 $Comp
-L power:GND #PWR?
+L power:GND #PWR0133
 U 1 1 62819CFA
 P 12850 6700
-F 0 "#PWR?" H 12850 6450 50  0001 C CNN
+F 0 "#PWR0133" H 12850 6450 50  0001 C CNN
 F 1 "GND" H 12855 6527 50  0000 C CNN
 F 2 "" H 12850 6700 50  0001 C CNN
@@
 $EndComp
 $Comp
-L Device:R_Pack08 RN?
+L Device:R_Pack08 RN206
 U 1 1 62819D01
 P 12550 6500
-F 0 "RN?" H 12938 6546 50  0000 L CNN
+F 0 "RN206" H 12938 6546 50  0000 L CNN
 F 1 "330 x 8" H 12938 6455 50  0000 L CNN
 F 2 "Package_DIP:DIP-16_W7.62mm_Socket" V 13025 6500 50  0001 C CNN
@@
 	13900 5950 13900 6300
 $Comp
-L Device:R_Pack08_Split RN?
+L Device:R_Pack08_Split RN201
 U 1 1 631A0905
 P 6600 1850
-F 0 "RN?" H 6688 1896 50  0000 L CNN
+F 0 "RN201" H 6688 1896 50  0000 L CNN
 F 1 "330 x 8" H 6688 1805 50  0000 L CNN
 F 2 "Package_DIP:DIP-16_W7.62mm_Socket" V 6520 1850 50  0001 C CNN
@@
 $EndComp
 $Comp
-L Device:R_Pack08_Split RN?
-U 2 1 634E3540
+L Device:R_Pack08_Split RN201
+U 5 1 634E3540
 P 7600 1850
-F 0 "RN?" H 7688 1896 50  0000 L CNN
+F 0 "RN201" H 7688 1896 50  0000 L CNN
 F 1 "330 x 8" H 7688 1805 50  0000 L CNN
 F 2 "Package_DIP:DIP-16_W7.62mm_Socket" V 7520 1850 50  0001 C CNN
 F 3 "~" H 7600 1850 50  0001 C CNN
 F 4 "652-4116R-1-330" H 7600 1850 50  0001 C CNN "Mouser"
-	2    7600 1850
-	1    0    0    -1
-$EndComp
-$Comp
-L Device:R_Pack08_Split RN?
-U 3 1 634E3A49
+	5    7600 1850
+	1    0    0    -1
+$EndComp
+$Comp
+L Device:R_Pack08_Split RN202
+U 1 1 634E3A49
 P 8600 1850
-F 0 "RN?" H 8688 1896 50  0000 L CNN
+F 0 "RN202" H 8688 1896 50  0000 L CNN
 F 1 "330 x 8" H 8688 1805 50  0000 L CNN
 F 2 "Package_DIP:DIP-16_W7.62mm_Socket" V 8520 1850 50  0001 C CNN
 F 3 "~" H 8600 1850 50  0001 C CNN
 F 4 "652-4116R-1-330" H 8600 1850 50  0001 C CNN "Mouser"
-	3    8600 1850
-	1    0    0    -1
-$EndComp
-$Comp
-L Device:R_Pack08_Split RN?
-U 4 1 634E3F52
+	1    8600 1850
+	1    0    0    -1
+$EndComp
+$Comp
+L Device:R_Pack08_Split RN202
+U 5 1 634E3F52
 P 9600 1850
-F 0 "RN?" H 9688 1896 50  0000 L CNN
+F 0 "RN202" H 9688 1896 50  0000 L CNN
 F 1 "330 x 8" H 9688 1805 50  0000 L CNN
 F 2 "Package_DIP:DIP-16_W7.62mm_Socket" V 9520 1850 50  0001 C CNN
 F 3 "~" H 9600 1850 50  0001 C CNN
 F 4 "652-4116R-1-330" H 9600 1850 50  0001 C CNN "Mouser"
-	4    9600 1850
+	5    9600 1850
 	1    0    0    -1
 $EndComp
@@
 	9300 2400 8950 2400
 $Comp
-L Device:R_Pack08_Split RN?
-U 5 1 63BCD470
+L Device:R_Pack08_Split RN201
+U 2 1 63BCD470
 P 6600 4350
-F 0 "RN?" H 6688 4396 50  0000 L CNN
+F 0 "RN201" H 6688 4396 50  0000 L CNN
 F 1 "330 x 8" H 6688 4305 50  0000 L CNN
 F 2 "Package_DIP:DIP-16_W7.62mm_Socket" V 6520 4350 50  0001 C CNN
 F 3 "~" H 6600 4350 50  0001 C CNN
 F 4 "652-4116R-1-330" H 6600 4350 50  0001 C CNN "Mouser"
-	5    6600 4350
-	1    0    0    -1
-$EndComp
-$Comp
-L Device:R_Pack08_Split RN?
+	2    6600 4350
+	1    0    0    -1
+$EndComp
+$Comp
+L Device:R_Pack08_Split RN201
 U 6 1 63BCD477
 P 7600 4350
-F 0 "RN?" H 7688 4396 50  0000 L CNN
+F 0 "RN201" H 7688 4396 50  0000 L CNN
 F 1 "330 x 8" H 7688 4305 50  0000 L CNN
 F 2 "Package_DIP:DIP-16_W7.62mm_Socket" V 7520 4350 50  0001 C CNN
@@
 $EndComp
 $Comp
-L Device:R_Pack08_Split RN?
-U 7 1 63BCD47E
+L Device:R_Pack08_Split RN202
+U 2 1 63BCD47E
 P 8600 4350
-F 0 "RN?" H 8688 4396 50  0000 L CNN
+F 0 "RN202" H 8688 4396 50  0000 L CNN
 F 1 "330 x 8" H 8688 4305 50  0000 L CNN
 F 2 "Package_DIP:DIP-16_W7.62mm_Socket" V 8520 4350 50  0001 C CNN
 F 3 "~" H 8600 4350 50  0001 C CNN
 F 4 "652-4116R-1-330" H 8600 4350 50  0001 C CNN "Mouser"
-	7    8600 4350
-	1    0    0    -1
-$EndComp
-$Comp
-L Device:R_Pack08_Split RN?
-U 8 1 63BCD485
+	2    8600 4350
+	1    0    0    -1
+$EndComp
+$Comp
+L Device:R_Pack08_Split RN202
+U 6 1 63BCD485
 P 9600 4350
-F 0 "RN?" H 9688 4396 50  0000 L CNN
+F 0 "RN202" H 9688 4396 50  0000 L CNN
 F 1 "330 x 8" H 9688 4305 50  0000 L CNN
 F 2 "Package_DIP:DIP-16_W7.62mm_Socket" V 9520 4350 50  0001 C CNN
 F 3 "~" H 9600 4350 50  0001 C CNN
 F 4 "652-4116R-1-330" H 9600 4350 50  0001 C CNN "Mouser"
-	8    9600 4350
+	6    9600 4350
 	1    0    0    -1
 $EndComp
@@
 	9300 4900 8950 4900
 $Comp
-L Device:R_Pack08_Split RN?
-U 1 1 647F8913
+L Device:R_Pack08_Split RN201
+U 3 1 647F8913
 P 6600 6850
-F 0 "RN?" H 6688 6896 50  0000 L CNN
+F 0 "RN201" H 6688 6896 50  0000 L CNN
 F 1 "330 x 8" H 6688 6805 50  0000 L CNN
 F 2 "Package_DIP:DIP-16_W7.62mm_Socket" V 6520 6850 50  0001 C CNN
 F 3 "~" H 6600 6850 50  0001 C CNN
 F 4 "652-4116R-1-330" H 6600 6850 50  0001 C CNN "Mouser"
-	1    6600 6850
-	1    0    0    -1
-$EndComp
-$Comp
-L Device:R_Pack08_Split RN?
-U 2 1 647F891A
+	3    6600 6850
+	1    0    0    -1
+$EndComp
+$Comp
+L Device:R_Pack08_Split RN201
+U 7 1 647F891A
 P 7600 6850
-F 0 "RN?" H 7688 6896 50  0000 L CNN
+F 0 "RN201" H 7688 6896 50  0000 L CNN
 F 1 "330 x 8" H 7688 6805 50  0000 L CNN
 F 2 "Package_DIP:DIP-16_W7.62mm_Socket" V 7520 6850 50  0001 C CNN
 F 3 "~" H 7600 6850 50  0001 C CNN
 F 4 "652-4116R-1-330" H 7600 6850 50  0001 C CNN "Mouser"
-	2    7600 6850
-	1    0    0    -1
-$EndComp
-$Comp
-L Device:R_Pack08_Split RN?
+	7    7600 6850
+	1    0    0    -1
+$EndComp
+$Comp
+L Device:R_Pack08_Split RN202
 U 3 1 647F8921
 P 8600 6850
-F 0 "RN?" H 8688 6896 50  0000 L CNN
+F 0 "RN202" H 8688 6896 50  0000 L CNN
 F 1 "330 x 8" H 8688 6805 50  0000 L CNN
 F 2 "Package_DIP:DIP-16_W7.62mm_Socket" V 8520 6850 50  0001 C CNN
@@
 $EndComp
 $Comp
-L Device:R_Pack08_Split RN?
-U 4 1 647F8928
+L Device:R_Pack08_Split RN202
+U 7 1 647F8928
 P 9600 6850
-F 0 "RN?" H 9688 6896 50  0000 L CNN
+F 0 "RN202" H 9688 6896 50  0000 L CNN
 F 1 "330 x 8" H 9688 6805 50  0000 L CNN
 F 2 "Package_DIP:DIP-16_W7.62mm_Socket" V 9520 6850 50  0001 C CNN
 F 3 "~" H 9600 6850 50  0001 C CNN
 F 4 "652-4116R-1-330" H 9600 6850 50  0001 C CNN "Mouser"
-	4    9600 6850
+	7    9600 6850
 	1    0    0    -1
 $EndComp
@@
 	9300 7400 8900 7400
 $Comp
-L Device:R_Pack08_Split RN?
-U 5 1 64F9E62B
+L Device:R_Pack08_Split RN201
+U 4 1 64F9E62B
 P 6600 9350
-F 0 "RN?" H 6688 9396 50  0000 L CNN
+F 0 "RN201" H 6688 9396 50  0000 L CNN
 F 1 "330 x 8" H 6688 9305 50  0000 L CNN
 F 2 "Package_DIP:DIP-16_W7.62mm_Socket" V 6520 9350 50  0001 C CNN
 F 3 "~" H 6600 9350 50  0001 C CNN
 F 4 "652-4116R-1-330" H 6600 9350 50  0001 C CNN "Mouser"
-	5    6600 9350
-	1    0    0    -1
-$EndComp
-$Comp
-L Device:R_Pack08_Split RN?
-U 6 1 64F9E632
+	4    6600 9350
+	1    0    0    -1
+$EndComp
+$Comp
+L Device:R_Pack08_Split RN201
+U 8 1 64F9E632
 P 7600 9350
-F 0 "RN?" H 7688 9396 50  0000 L CNN
+F 0 "RN201" H 7688 9396 50  0000 L CNN
 F 1 "330 x 8" H 7688 9305 50  0000 L CNN
 F 2 "Package_DIP:DIP-16_W7.62mm_Socket" V 7520 9350 50  0001 C CNN
 F 3 "~" H 7600 9350 50  0001 C CNN
 F 4 "652-4116R-1-330" H 7600 9350 50  0001 C CNN "Mouser"
-	6    7600 9350
-	1    0    0    -1
-$EndComp
-$Comp
-L Device:R_Pack08_Split RN?
-U 7 1 64F9E639
+	8    7600 9350
+	1    0    0    -1
+$EndComp
+$Comp
+L Device:R_Pack08_Split RN202
+U 4 1 64F9E639
 P 8600 9350
-F 0 "RN?" H 8688 9396 50  0000 L CNN
+F 0 "RN202" H 8688 9396 50  0000 L CNN
 F 1 "330 x 8" H 8688 9305 50  0000 L CNN
 F 2 "Package_DIP:DIP-16_W7.62mm_Socket" V 8520 9350 50  0001 C CNN
 F 3 "~" H 8600 9350 50  0001 C CNN
 F 4 "652-4116R-1-330" H 8600 9350 50  0001 C CNN "Mouser"
-	7    8600 9350
-	1    0    0    -1
-$EndComp
-$Comp
-L Device:R_Pack08_Split RN?
+	4    8600 9350
+	1    0    0    -1
+$EndComp
+$Comp
+L Device:R_Pack08_Split RN202
 U 8 1 64F9E640
 P 9600 9350
-F 0 "RN?" H 9688 9396 50  0000 L CNN
+F 0 "RN202" H 9688 9396 50  0000 L CNN
 F 1 "330 x 8" H 9688 9305 50  0000 L CNN
 F 2 "Package_DIP:DIP-16_W7.62mm_Socket" V 9520 9350 50  0001 C CNN
@@
 Wire Wire Line
 	9300 9900 8900 9900
+Connection ~ 12850 3400
 $EndSCHEMATC
