File: design-files/clock-module/clock-module.sch (KiCad schematic (older format))
At the start: 32 parts, among them J101 CUI_PJ-097BH-5_5-2_5mm-5A, Q101 2N6491, SW101 SW_Push, SW102 SW_SPDT, SW103 SW_SPDT, U101 NE555P, U102 NE555P, U103 NE555P, U104 74HCT00, U105 74HCT00

Commit message: Change to 5mm LS ceramic caps.
Parts:
- C101, C102, C104, C105, C106, C107, C108, C109, C110: footprint Capacitor_THT:C_Radial_D6.3mm_H5.0mm_P2.50mm -> Capacitor_THT:C_Disc_D4.7mm_W2.5mm_P5.00mm
- J101: Mouser (none) -> 490-PJ-079BH
Changed lines of the file:
@@
 F 0 "C101" H 2592 1696 50  0000 L CNN
 F 1 "0.1µF" H 2592 1605 50  0000 L CNN
-F 2 "Capacitor_THT:C_Radial_D6.3mm_H5.0mm_P2.50mm" H 2500 1650 50  0001 C CNN
+F 2 "Capacitor_THT:C_Disc_D4.7mm_W2.5mm_P5.00mm" H 2500 1650 50  0001 C CNN
 F 3 "~" H 2500 1650 50  0001 C CNN
 F 4 "80-C320C104K2R5TA" H 2500 1650 50  0001 C CNN "Mouser"
@@
 F 0 "C107" H 8342 1696 50  0000 L CNN
 F 1 "0.1µF" H 8342 1605 50  0000 L CNN
-F 2 "Capacitor_THT:C_Radial_D6.3mm_H5.0mm_P2.50mm" H 8250 1650 50  0001 C CNN
+F 2 "Capacitor_THT:C_Disc_D4.7mm_W2.5mm_P5.00mm" H 8250 1650 50  0001 C CNN
 F 3 "~" H 8250 1650 50  0001 C CNN
 F 4 "80-C320C104K2R5TA" H 8250 1650 50  0001 C CNN "Mouser"
@@
 F 0 "C102" H 1050 2950 50  0000 L CNN
 F 1 "0.01µF" H 950 2850 50  0000 L CNN
-F 2 "Capacitor_THT:C_Radial_D6.3mm_H5.0mm_P2.50mm" H 1350 2900 50  0001 C CNN
+F 2 "Capacitor_THT:C_Disc_D4.7mm_W2.5mm_P5.00mm" H 1350 2900 50  0001 C CNN
 F 3 "~" H 1350 2900 50  0001 C CNN
 F 4 "80-C315C103K5R-TR" H 1350 2900 50  0001 C CNN "Mouser"
@@
 F 0 "C105" H 4400 2950 50  0000 L CNN
 F 1 "0.01µF" H 4400 2850 50  0000 L CNN
-F 2 "Capacitor_THT:C_Radial_D6.3mm_H5.0mm_P2.50mm" H 4300 2900 50  0001 C CNN
+F 2 "Capacitor_THT:C_Disc_D4.7mm_W2.5mm_P5.00mm" H 4300 2900 50  0001 C CNN
 F 3 "~" H 4300 2900 50  0001 C CNN
 F 4 "80-C315C103K5R-TR" H 4300 2900 50  0001 C CNN "Mouser"
@@
 F 0 "C106" H 5900 2950 50  0000 L CNN
 F 1 "0.1µF" H 5900 2850 50  0000 L CNN
-F 2 "Capacitor_THT:C_Radial_D6.3mm_H5.0mm_P2.50mm" H 5800 2900 50  0001 C CNN
+F 2 "Capacitor_THT:C_Disc_D4.7mm_W2.5mm_P5.00mm" H 5800 2900 50  0001 C CNN
 F 3 "~" H 5800 2900 50  0001 C CNN
 F 4 "80-C320C104K2R5TA" H 5800 2900 50  0001 C CNN "Mouser"
@@
 F 0 "C104" H 5100 1700 50  0000 L CNN
 F 1 "0.1µF" H 5100 1600 50  0000 L CNN
-F 2 "Capacitor_THT:C_Radial_D6.3mm_H5.0mm_P2.50mm" H 5400 1650 50  0001 C CNN
+F 2 "Capacitor_THT:C_Disc_D4.7mm_W2.5mm_P5.00mm" H 5400 1650 50  0001 C CNN
 F 3 "~" H 5400 1650 50  0001 C CNN
 F 4 "80-C320C104K2R5TA" H 5400 1650 50  0001 C CNN "Mouser"
@@
 F 0 "C108" H 7250 2950 50  0000 L CNN
 F 1 "0.01µF" H 7250 2850 50  0000 L CNN
-F 2 "Capacitor_THT:C_Radial_D6.3mm_H5.0mm_P2.50mm" H 7150 2900 50  0001 C CNN
+F 2 "Capacitor_THT:C_Disc_D4.7mm_W2.5mm_P5.00mm" H 7150 2900 50  0001 C CNN
 F 3 "~" H 7150 2900 50  0001 C CNN
 F 4 "80-C315C103K5R-TR" H 7150 2900 50  0001 C CNN "Mouser"
@@
 F 0 "C109" H 7250 3950 50  0000 L CNN
 F 1 "0.1µF" H 7250 3850 50  0000 L CNN
-F 2 "Capacitor_THT:C_Radial_D6.3mm_H5.0mm_P2.50mm" H 7550 3900 50  0001 C CNN
+F 2 "Capacitor_THT:C_Disc_D4.7mm_W2.5mm_P5.00mm" H 7550 3900 50  0001 C CNN
 F 3 "~" H 7550 3900 50  0001 C CNN
 F 4 "80-C320C104K2R5TA" H 7550 3900 50  0001 C CNN "Mouser"
@@
 F 0 "C110" H 8200 3950 50  0000 L CNN
 F 1 "0.1µF" H 8200 3850 50  0000 L CNN
-F 2 "Capacitor_THT:C_Radial_D6.3mm_H5.0mm_P2.50mm" H 8500 3900 50  0001 C CNN
+F 2 "Capacitor_THT:C_Disc_D4.7mm_W2.5mm_P5.00mm" H 8500 3900 50  0001 C CNN
 F 3 "~" H 8500 3900 50  0001 C CNN
 F 4 "80-C320C104K2R5TA" H 8500 3900 50  0001 C CNN "Mouser"
@@
 F 2 "jrt-Connectors:CUI_PJ-097BH-5_5-2_5mm-5A" H 4200 6200 50  0001 C CNN
 F 3 "" H 4200 6200 50  0001 C CNN
+F 4 "490-PJ-079BH" H 4000 6300 50  0001 C CNN "Mouser"
 	1    4000 6300
 	1    0    0    -1
